File: KiCAD filer/Kretsschema/Rasppipico för HAN-port.kicad_sch (KiCad schematic)
At the start: 3 parts, among them J1 RJ12

Commit message: Updaterar filer för PCB.
Fixade storleken på motståndet.
Parts:
- R1: footprint Resistor_THT:R_Axial_DIN0614_L14.3mm_D5.7mm_P20.32mm_Horizontal -> Resistor_THT:R_Axial_DIN0207_L6.3mm_D2.5mm_P10.16mm_Horizontal
Changed lines of the file:
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@@
 			)
 		)
-		(property "Footprint" "Resistor_THT:R_Axial_DIN0614_L14.3mm_D5.7mm_P20.32mm_Horizontal"
+		(property "Footprint" "Resistor_THT:R_Axial_DIN0207_L6.3mm_D2.5mm_P10.16mm_Horizontal"
 			(at 146.812 66.04 90)
 			(effects
